File: 08. VUmeter/Electronics/VUmeter_PCB/VUmeter_PCB.kicad_sch (KiCad schematic)
At the start: 4 parts, among them J1 Screw_Terminal_01x09, J2 Screw_Terminal_01x09, J3 Screw_Terminal_01x03, J4 Screw_Terminal_01x03

Commit message: 08. VUmeter. Start PCB proyect.
Parts:
- added J5: Tira LED, Connector_PinHeader_2.54mm:PinHeader_1x03_P2.54mm_Vertical, symbol Connector:Screw_Terminal_01x03
- added J6: Alimentacion, Connector_PinHeader_2.54mm:PinHeader_1x02_P2.54mm_Vertical, symbol Connector:Screw_Terminal_01x02
- J1: value Screw_Terminal_01x09 -> ESP32S3 SuperMini I; footprint (none) -> Connector_PinHeader_2.54mm:PinHeader_1x09_P2.54mm_Vertical
- J2: value Screw_Terminal_01x09 -> ESP32S3 SuperMini D; footprint (none) -> Connector_PinHeader_2.54mm:PinHeader_1x09_P2.54mm_Vertical
- J3: value Screw_Terminal_01x03 -> INMP4144 I; footprint (none) -> Connector_PinHeader_2.54mm:PinHeader_1x03_P2.54mm_Vertical
- J4: value Screw_Terminal_01x03 -> INMP4144 D; footprint (none) -> Connector_PinHeader_2.54mm:PinHeader_1x03_P2.54mm_Vertical
Connections:
- net 10: now also J3.1 (Pin_1)
- net 11: now also J4.2 (Pin_2)
- net 12: now also J4.3 (Pin_3)
- net 13: now also J5.2 (Pin_2)
- net 3V3: now also J3.2 (Pin_2)
- net 5V: now also J5.1 (Pin_1), J6.2 (Pin_2)
- net GND: now also J3.3 (Pin_3), J4.1 (Pin_1), J5.3 (Pin_3), J6.1 (Pin_1)
Other:
- moved on the sheet: J4

Commit message: 08.VUmeter. PCB update and Software update according to schematic.
Parts:
- removed J6: Alimentacion, Connector_PinHeader_2.54mm:PinHeader_1x02_P2.54mm_Vertical, symbol Connector:Screw_Terminal_01x02
Connections:
- net 10: now also J5.3 (Pin_3); no longer J3.1 (Pin_1)
- net 11: now also J3.1 (Pin_1); no longer J4.2 (Pin_2)
- net 13: now also J4.2 (Pin_2); no longer J5.2 (Pin_2)
- net GND: now also J5.2 (Pin_2); no longer J5.3 (Pin_3)
Changed lines of the file:
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@@
-	(wire
-		(pts
-			(xy 217.17 74.93) (xy 222.25 74.93)
-		)
-		(stroke
-			(width 0)
-			(type default)
-		)
-	)
 	(wire
 		(pts
@@
 	(wire
 		(pts
-			(xy 190.5 99.06) (xy 207.01 99.06)
-		)
-		(stroke
-			(width 0)
-			(type default)
-		)
-	)
-	(wire
-		(pts
 			(xy 190.5 104.14) (xy 196.85 104.14)
 		)
@@
 	(wire
 		(pts
+			(xy 190.5 99.06) (xy 196.85 99.06)
+		)
+		(stroke
+			(width 0)
+			(type default)
+		)
+	)
+	(wire
+		(pts
 			(xy 142.24 86.36) (xy 148.59 86.36)
 		)
@@
 	(wire
 		(pts
-			(xy 217.17 77.47) (xy 222.25 77.47)
-		)
-		(stroke
-			(width 0)
-			(type default)
-		)
-	)
-	(wire
-		(pts
-			(xy 190.5 91.44) (xy 196.85 91.44)
+			(xy 190.5 91.44) (xy 207.01 91.44)
 		)
 		(stroke
@@
 		)
 	)
-	(label "13"
-		(at 217.17 86.36 0)
-		(fields_autoplaced yes)
-		(effects
-			(font
-				(size 1.27 1.27)
-			)
-			(justify left bottom)
-		)
-	)
 	(label "8"
 		(at 196.85 104.14 0)
@@
 		)
 	)
+	(label "SD"
+		(at 207.01 96.52 0)
+		(fields_autoplaced yes)
+		(effects
+			(font
+				(size 1.27 1.27)
+			)
+			(justify left bottom)
+		)
+	)
 	(label "RX"
 		(at 142.24 86.36 0)
@@
 		)
 	)
-	(label "SD"
-		(at 207.01 99.06 0)
-		(fields_autoplaced yes)
-		(effects
-			(font
-				(size 1.27 1.27)
-			)
-			(justify left bottom)
-		)
-	)
-	(label "GND"
-		(at 217.17 74.93 0)
-		(fields_autoplaced yes)
-		(effects
-			(font
-				(size 1.27 1.27)
-			)
-			(justify left bottom)
-		)
-	)
 	(label "WS"
 		(at 195.58 118.11 0)
@@
 		)
 	)
+	(label "WS"
+		(at 207.01 91.44 0)
+		(fields_autoplaced yes)
+		(effects
+			(font
+				(size 1.27 1.27)
+			)
+			(justify left bottom)
+		)
+	)
 	(label "SCK"
 		(at 207.01 93.98 0)
@@
 		)
 	)
-	(label "5V"
-		(at 217.17 77.47 0)
-		(fields_autoplaced yes)
-		(effects
-			(font
-				(size 1.27 1.27)
-			)
-			(justify left bottom)
-		)
-	)
-	(label "GND"
-		(at 217.17 88.9 0)
-		(fields_autoplaced yes)
-		(effects
-			(font
-				(size 1.27 1.27)
-			)
-			(justify left bottom)
-		)
-	)
 	(label "GND"
 		(at 201.93 120.65 0)
@@
 		)
 	)
+	(label "10"
+		(at 217.17 88.9 0)
+		(fields_autoplaced yes)
+		(effects
+			(font
+				(size 1.27 1.27)
+			)
+			(justify left bottom)
+		)
+	)
 	(label "9"
 		(at 196.85 101.6 0)
@@
 		)
 	)
+	(label "GND"
+		(at 217.17 86.36 0)
+		(fields_autoplaced yes)
+		(effects
+			(font
+				(size 1.27 1.27)
+			)
+			(justify left bottom)
+		)
+	)
 	(label "3"
 		(at 142.24 93.98 0)
-		(fields_autoplaced yes)
-		(effects
-			(font
-				(size 1.27 1.27)
-			)
-			(justify left bottom)
-		)
-	)
-	(label "WS"
-		(at 207.01 96.52 0)
 		(fields_autoplaced yes)
 		(effects
@@
 					(unit 1)
 				)
-			)
-		)
-	)
-	(symbol
-		(lib_id "Connector:Screw_Terminal_01x02")
-		(at 227.33 74.93 0)
-		(unit 1)
-		(exclude_from_sim no)
-		(in_bom yes)
-		(on_board yes)
-		(dnp no)
-		(fields_autoplaced yes)
-		(property "Reference" "J6"
-			(at 229.87 74.9299 0)
-			(effects
-				(font
-					(size 1.27 1.27)
-				)
-				(justify left)
-			)
-		)
-		(property "Value" "Alimentacion"
-			(at 229.87 77.4699 0)
-			(effects
-				(font
-					(size 1.27 1.27)
-				)
-				(justify left)
-			)
-		)
-		(property "Footprint" "Connector_PinHeader_2.54mm:PinHeader_1x02_P2.54mm_Vertical"
-			(at 227.33 74.93 0)
-			(effects
-				(font
-					(size 1.27 1.27)
-				)
-				(hide yes)
-			)
-		)
-		(property "Datasheet" "~"
-			(at 227.33 74.93 0)
-			(effects
-				(font
-					(size 1.27 1.27)
-				)
-				(hide yes)
-			)
-		)
-		(property "Description" "Generic screw terminal, single row, 01x02, script generated (kicad-library-utils/schlib/autogen/connector/)"
-			(at 227.33 74.93 0)
-			(effects
-				(font
-					(size 1.27 1.27)
-				)
-				(hide yes)
-			)
-		)
-		(pin "2"
-		)
-		(pin "1"
-		)
-		(instances
-			(project "VUmeter_PCB"
-				(path "/e78c4d2b-e79a-4dfc-8f19-81c3792a8ef1"
-					(reference "J6")
-					(unit 1)
-				)
